Commit message: feat : change CoM of the unknown obj

File: rsc/slope/slope.urdf (robot description, URDF)
Before this commit: robot slope, 1 links, 1 joints
Links:
- added link base; visual box size=0.001 0.001 0.001
- link base_link: geometry collision mesh filename=slope.obj scale=1 1 1; visual mesh filename=/Users/yushin/raisim_workspace/raisimExample/rsc/slope/slop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 scale=1 1 1
Joints:
- joint fixed_joint: parent world -> base
